File: Analog_LFR.kicad_sch (KiCad schematic)
At the start: 134 parts, among them Q1 AO3400A, Q2 AO3400A, U1 MCP6004T-I/SL, U2 MCP6004T-I/SL, U3 MCP6004T-I/SL, U4 MCP6004T-I/SL, U5 MCP6004T-I/SL, U6 MCP6004T-I/SL, U7 MCP6004T-I/SL, U8 LM339, U9 AP63205WU

Commit message: Gate pull up changed for faster switching
Parts:
- R211, R212: value 4.7K -> 2.2K

Commit message: ERROR WEIGHTS FIXED
Parts:
- R402, R407: value 100K -> 20K
- R403, R408: value 51K -> 24K
- R405, R410: value 24K -> 51K
- R406, R411: value 20K -> 100K
Changed lines of the file:
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@@
 			)
 		)
-		(property "Value" "100K"
+		(property "Value" "20K"
 			(at 223.52 78.74 90)
 			(show_name no)
@@
 			)
 		)
-		(property "Value" "51K"
+		(property "Value" "24K"
 			(at 242.57 87.63 90)
 			(show_name no)
@@
 			)
 		)
-		(property "Value" "24K"
+		(property "Value" "51K"
 			(at 242.57 105.41 90)
 			(show_name no)
@@
 			)
 		)
-		(property "Value" "20K"
+		(property "Value" "100K"
 			(at 242.57 115.57 90)
 			(show_name no)
@@
 			)
 		)
-		(property "Value" "20K"
+		(property "Value" "100K"
 			(at 223.52 115.57 90)
 			(show_name no)
@@
 			)
 		)
-		(property "Value" "100K"
+		(property "Value" "20K"
 			(at 242.57 78.74 90)
 			(show_name no)
@@
 			)
 		)
-		(property "Value" "24K"
+		(property "Value" "51K"
 			(at 223.52 105.41 90)
 			(show_name no)
@@
 			)
 		)
-		(property "Value" "51K"
+		(property "Value" "24K"
 			(at 223.52 87.63 90)
 			(show_name no)
