File: Anlog_LFR.kicad_pcb (KiCad board)
At the start: 4 copper layers, 99.6 x 98.3 mm, 148 parts, among them Q1 AO3400A, Q2 AO3400A, U1 MCP6004T-I/SL, U2 MCP6004T-I/SL, U3 MCP6004T-I/SL, U4 MCP6004T-I/SL, U5 MCP6004T-I/SL, U6 MCP6004T-I/SL, U7 MCP6004T-I/SL, U8 LM339, U9 AP63205WU

Commit message: ERROR WEIGHTS FIXED
Parts:
- R211, R212: value 4.7K -> 2.2K
- R402, R407: value 100K -> 20K
- R403, R408: value 51K -> 24K
- R405, R410: value 24K -> 51K
- R406, R411: value 20K -> 100K
